File: GTI_V4_KiCad/GTI_V4_KiCad.kicad_sch (KiCad schematic)
At the start: 141 parts, among them IC1 MASTERGAN2TR, IC2 MASTERGAN2TR, IC3 MAX253CSA+, IC4 AMC1306M25QDWVRQ1, IC5 AMC1306M25QDWVRQ1, IC6 AMC1306M25QDWVRQ1, IC7 MAX253CSA+, IC8 MAX253CSA+, IC9 AMC1306M25QDWVRQ1, J1 Screw_Terminal_01x03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

Commit message: Add files via upload
Parts:
- added C59: 1uF, Capacitor_SMD:C_0603_1608Metric, symbol Device:C
- added C69: 100nF, Capacitor_SMD:C_0603_1608Metric, symbol Device:C
Connections:
- net +3.3V: now also C59.1, C69.1
- net GNDD: now also C59.2, C69.2
Other:
- moved on the sheet: C1, C10, C16, C17, C18, C19, C2, C21, C3, C4, D4, J4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

Commit message: 99% finished PCB
Parts:
- added C70: 100nF, Capacitor_SMD:C_0603_1608Metric, symbol Device:C
- added C71: 10nF, Capacitor_SMD:C_0603_1608Metric, symbol Device:C
Connections:
- net +3.3V: now also J4.1 (Pin_1), C70.1
- net GNDD: now also J4.3 (Pin_3), C70.2, C71.2; no longer J4.6 (Pin_6)
- net NRST: now also J4.5 (Pin_5)
- net VCC: now also C71.1
- net JTCK-SWCLK renamed SWCLK
- net JTDI: no longer names the net of U1.50 (PA15)
- net JTDI: no longer J4.3 (Pin_3)
- net JTDO-TRACESWO renamed SWDIO
- net SWDIO: now also U1.46 (PA13); no longer U1.55 (PB3)
- removed net JTMS-SWDIO: J4.1 (Pin_1), U1.46 (PA13)
- net NJTRST: no longer names the net of U1.56 (PB4)
- net NJTRST: no longer J4.5 (Pin_5)
- new net SWO: J4.6 (Pin_6), U1.55 (PB3)

Commit message: The finished and used PCB
Parts:
- C25: value 1uF -> 4.7uF
- C71: value 10nF -> 1uF
- R7: value 2.2R -> 6.8R
Changed lines of the file:
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@@
       (effects (font (size 1.27 1.27)) (justify left))
     )
-    (property "Value" "1uF" (id 1) (at 194.31 106.68 0)
+    (property "Value" "4.7uF" (id 1) (at 194.31 106.68 0)
       (effects (font (size 1.27 1.27)) (justify left))
     )
@@
       (effects (font (size 1.27 1.27)) (justify left))
     )
-    (property "Value" "10nF" (id 1) (at 304.8 137.16 0)
+    (property "Value" "1uF" (id 1) (at 304.8 137.16 0)
       (effects (font (size 1.27 1.27)) (justify left))
     )
@@
   (symbol (lib_id "power:+3.3V") (at 44.45 101.6 0) (unit 1)
     (in_bom yes) (on_board yes) (fields_autoplaced)
-    (property "Reference" "#PWR?" (id 0) (at 44.45 105.41 0)
+    (property "Reference" "#PWR0115" (id 0) (at 44.45 105.41 0)
       (effects (font (size 1.27 1.27)) hide)
     )
@@
       (effects (font (size 1.27 1.27)) (justify left))
     )
-    (property "Value" "2.2R" (id 1) (at 288.798 89.3322 0)
+    (property "Value" "6.8R" (id 1) (at 288.798 89.3322 0)
       (effects (font (size 1.27 1.27)) (justify left))
     )
@@
       (reference "#PWR0114") (unit 1) (value "GNDD") (footprint "")
     )
+    (path "/844abd9b-b350-4544-902c-40e4b8f21f3c"
+      (reference "#PWR0115") (unit 1) (value "+3.3V") (footprint "")
+    )
     (path "/2d088de9-a606-491f-b18a-63e4604a3193"
       (reference "#PWR0117") (unit 1) (value "VBUS") (footprint "")
@@
       (reference "#PWR0123") (unit 1) (value "GND") (footprint "")
     )
-    (path "/844abd9b-b350-4544-902c-40e4b8f21f3c"
-      (reference "#PWR?") (unit 1) (value "+3.3V") (footprint "")
-    )
     (path "/c46dcd28-fc11-4708-aa27-66df842f6468"
       (reference "C1") (unit 1) (value "100nF") (footprint "Capacitor_SMD:C_0603_1608Metric")
@@
     )
     (path "/022f31cb-900a-4d06-b79c-6e6698b498b2"
-      (reference "C25") (unit 1) (value "1uF") (footprint "Capacitor_SMD:C_0603_1608Metric")
+      (reference "C25") (unit 1) (value "4.7uF") (footprint "Capacitor_SMD:C_0603_1608Metric")
     )
     (path "/10d4c2f2-33e3-45f0-9582-244e74e1423b"
@@
     )
     (path "/633deeef-0ade-4329-b819-d915dc6fc9ed"
-      (reference "C71") (unit 1) (value "10nF") (footprint "Capacitor_SMD:C_0603_1608Metric")
+      (reference "C71") (unit 1) (value "1uF") (footprint "Capacitor_SMD:C_0603_1608Metric")
     )
     (path "/951b7b55-2863-405e-ae6d-1fd17c3ec689"
@@
     )
     (path "/e4bf290b-a183-4fbe-880d-b39fd4cc4501"
-      (reference "R7") (unit 1) (value "2.2R") (footprint "Resistor_SMD:R_2512_6332Metric")
+      (reference "R7") (unit 1) (value "6.8R") (footprint "Resistor_SMD:R_2512_6332Metric")
     )
     (path "/14f76ad8-a66a-4187-a408-954b91a7b33c"
